File: lilyPad_RP2040/lilyPad_RP2040.kicad_sch (KiCad schematic)
At the start: 46 parts, among them J1 Conn_01x02, J10 Conn_01x01, J11 Conn_01x01, J12 Conn_01x01, J13 Conn_01x01, J14 Conn_01x01, J15 Conn_01x01, J16 Conn_01x01, J17 Conn_01x01, J18 Conn_01x01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

Commit message: fonoooo
Parts:
- added D1, D2: LED, LED_SMD:LED_0603_1608Metric, symbol Device:LED
- added R7, R8: 220, Resistor_SMD:R_0603_1608Metric, symbol Device:R
- Y1: value Crystal -> C9002; footprint (none) -> Crystal:Crystal_SMD_3225-4Pin_3.2x2.5mm; symbol Device:Crystal_GND23 -> Device:Crystal_GND24
Connections:
- net +3V3: now also D1.2 (A)
- net GND: now also C10.2, C9.2, Y1.4, R7.1, R8.1; no longer Y1.3
- net GPIO26_ADC0: now also J17.1 (Pin_1)
- net GPIO27_ADC1: now also J18.1 (Pin_1)
- net GPIO28_ADC2: now also J19.1 (Pin_1)
- net GPIO29_ADC3: now also D2.2 (A)
- net XIN: now also Y1.1; no longer Y1.4
- net at C13.2, R4.1: now also Y1.3; no longer Y1.1
- net GPIO13: no longer names the net of U1.16 (GPIO13)
- net GPIO13: no longer J17.1 (Pin_1)
- net GPIO14: no longer names the net of U1.17 (GPIO14)
- net GPIO14: no longer J18.1 (Pin_1)
- net GPIO15: no longer names the net of U1.18 (GPIO15)
- net GPIO15: no longer J19.1 (Pin_1)
- new net: D1.1 (K), R7.2
- new net: D2.1 (K), R8.2
- no-connect marks 12 -> 15
