File: lilyPad_RP2040/lilyPad_RP2040.kicad_pcb (KiCad board)
At the start: 2 copper layers, 50 x 50 mm, 47 parts, among them J1 Conn_01x02, J10 Conn_01x01, J11 Conn_01x01, J12 Conn_01x01, J13 Conn_01x01, J14 Conn_01x01, J15 Conn_01x01, J16 Conn_01x01, J17 Conn_01x01, J18 Conn_01x01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

Commit message: fonoooo
Parts:
- removed J22, J23: Conn_01x01, lilyPad:LilyPad_Pad
- added D1: LED, LED_SMD:LED_0603_1608Metric, F.Cu at (143.2, 77.6)
- added D2: LED, LED_SMD:LED_0603_1608Metric, F.Cu at (137.7, 82.2)
- added R7: 220, Resistor_SMD:R_0603_1608Metric, F.Cu at (143.2, 79.4)
- added R8: 220, Resistor_SMD:R_0603_1608Metric, F.Cu at (137.7, 83.9)
- added Y1: C9002, Crystal:Crystal_SMD_3225-4Pin_3.2x2.5mm, F.Cu at (135.2, 102.1)
- moved C4 117.1 mm to (138.1, 97.9)
- moved C5 115.8 mm to (138.7, 95.6)
- moved C15 113.9 mm to (146.0, 81.9)
- moved C3 113.7 mm to (137.5, 87.6), turned to 90 degrees
- moved C8 113.3 mm to (139.1, 87.6), turned to 90 degrees
- moved C13 113.2 mm to (138.2, 102.1), turned to 90 degrees
- moved C2 113.0 mm to (135.9, 87.6), turned to 90 degrees
- moved C1 112.5 mm to (134.3, 87.6), turned to 90 degrees
- moved C14 109.1 mm to (141.3, 81.9), turned to 180 degrees
- moved C12 108.7 mm to (132.2, 102.0), turned to 90 degrees
- moved R4 106.2 mm to (134.6, 99.5), turned to 180 degrees
- moved C10 104.2 mm to (131.9, 86.1), turned to 90 degrees
- moved R2 103.8 mm to (138.4, 77.5), turned to -117 degrees
- moved C9 103.6 mm to (130.3, 86.1), turned to 90 degrees
- moved R6 103.1 mm to (139.9, 78.2), turned to 63 degrees
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Connections:
- C10 pad 2: Net-(C10-Pad2) -> GND
- C9 pad 2: Net-(C10-Pad2) -> GND
- J17 pad 1: /GPIO13 -> /GPIO26_ADC0
- J18 pad 1: /GPIO14 -> /GPIO27_ADC1
- J19 pad 1: /GPIO15 -> /GPIO28_ADC2
- U1 pad 16: /GPIO13 -> unconnected-(U1-GPIO13-Pad16)
- U1 pad 17: /GPIO14 -> unconnected-(U1-GPIO14-Pad17)
- U1 pad 18: /GPIO15 -> unconnected-(U1-GPIO15-Pad18)
Routing:
- net +3V3: track 0.00 -> 116.8 mm, vias 0 -> 10
- net /GPIO0/TX0: track 0.00 -> 38.7 mm
- net /GPIO1/RX0: track 0.00 -> 34.7 mm
- net GND: track 0.00 -> 32.3 mm, vias 0 -> 22
- net /GPIO2: track 0.00 -> 31.2 mm
- net /GPIO3: track 0.00 -> 27.3 mm
- net /~{CS}: track 0.00 -> 25.3 mm
- net /GPIO4: track 0.00 -> 23.8 mm
- net /GPIO12: track 0.00 -> 21.5 mm
- net /GPIO28_ADC2: track 0.00 -> 20.5 mm
- net /GPIO5: track 0.00 -> 20.4 mm
- net /GPIO26_ADC0: track 0.00 -> 19.3 mm
- net /GPIO27_ADC1: track 0.00 -> 18.5 mm
- net /GPIO11: track 0.00 -> 18.4 mm
- net /IO3: track 0.00 -> 17.6 mm
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- added copper zone on B.Cu, net GND

Commit message: update
Parts:
- J10, J11, J12, J13, J14, J15, J16, J17, J18, J19, J20, J21, J4, J5, J6, J7, J8, J9: footprint lilyPad:LilyPad_Pad -> lilyPad_PadCustomM3:LilyPadCustomPadM3

Commit message: finish_hw
Parts:
- moved J14 17.5 mm to (149.3, 105.3), turned to -153 degrees
- moved J13 17.3 mm to (142.9, 107.4), turned to -171 degrees
- moved J15 17.3 mm to (154.7, 101.4), turned to -135 degrees
- moved J12 16.7 mm to (136.2, 107.4), turned to 171 degrees
- moved J16 16.6 mm to (158.7, 95.9), turned to -117 degrees
- moved J11 15.8 mm to (129.8, 105.3), turned to 153 degrees
- moved J17 15.5 mm to (160.8, 89.5), turned to -99 degrees
- moved J10 14.4 mm to (124.3, 101.4), turned to 135 degrees
- moved J18 14.1 mm to (160.8, 82.8), turned to -81 degrees
- moved J3 13.5 mm to (153.0, 86.8), turned to -8 degrees
- moved J9 12.7 mm to (120.4, 95.9), turned to 117 degrees
- moved R4 12.4 mm to (146.5, 95.9), turned to -153 degrees
- moved J19 12.3 mm to (158.7, 76.4), turned to -63 degrees
- moved C4 12.3 mm to (148.6, 91.5), turned to 27 degrees
- moved C6 12.2 mm to (135.3, 97.7), turned to -153 degrees
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Routing:
- net VBUS: track 2.25 -> 18.5 mm, vias 0 -> 2
- net /GPIO28_ADC2: track 20.5 -> 25.7 mm
- net +3V3: track 116.8 -> 120.2 mm, vias 10 -> 11
- net /SWCLK: track 11.7 -> 14.2 mm
- net /SWD: track 9.99 -> 8.50 mm
- net GND: track 32.3 -> 33.8 mm, vias 22 -> 24
- net /GPIO11: track 18.4 -> 19.7 mm, vias 0 -> 1
- net /GPIO4: track 23.8 -> 25.0 mm
- net /GPIO10: track 15.9 -> 17.0 mm, vias 0 -> 1
- net /GPIO12: track 21.5 -> 20.5 mm, vias 0 -> 1
- net /XOUT: track 3.36 -> 2.57 mm
- net /XIN: track 6.38 -> 7.06 mm
- net /~{CS}: track 25.3 -> 26.0 mm
- added copper zone on F.Cu, net GND
Other:
- board size 50 x 50 mm -> 50.4 x 50.4 mm
- board text added: "0"
- board text added: "1"
- board text added: "11"
- board text added: "2"
- board text added: "3"
- board text added: "3v3"
- board text added: "4"
- board text added: "5"
- board text added: "6"
- board text added: "7"
- board text added: "8"
- board text added: "9"
- board text added: "A0"
- board text added: "A1"
- board text added: "A2"
- board text added: "BOOT"
- board text added: "GND"
- board text added: "SWD"
- board text added: "lilyPad rp2040"

Commit message: some changes
Routing:
- net +3V3: track 120.2 -> 118.2 mm
Changed lines of the file:
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@@
 	)
 	(setup
+		(stackup
+			(layer "F.SilkS"
+				(type "Top Silk Screen")
+			)
+			(layer "F.Paste"
+				(type "Top Solder Paste")
+			)
+			(layer "F.Mask"
+				(type "Top Solder Mask")
+				(thickness 0.01)
+			)
+			(layer "F.Cu"
+				(type "copper")
+				(thickness 0.035)
+			)
+			(layer "dielectric 1"
+				(type "core")
+				(thickness 1.51)
+				(material "FR4")
+				(epsilon_r 4.5)
+				(loss_tangent 0.02)
+			)
+			(layer "B.Cu"
+				(type "copper")
+				(thickness 0.035)
+			)
+			(layer "B.Mask"
+				(type "Bottom Solder Mask")
+				(thickness 0.01)
+			)
+			(layer "B.Paste"
+				(type "Bottom Solder Paste")
+			)
+			(layer "B.SilkS"
+				(type "Bottom Silk Screen")
+			)
+			(copper_finish "None")
+			(dielectric_constraints no)
+		)
 		(pad_to_mask_clearance 0)
 		(allow_soldermask_bridges_in_footprints no)
@@
 		(tags "resistor")
 		(property "Reference" "R6"
-			(at 0 -1.43 270)
+			(at 0 -1.43 -90)
 			(layer "F.SilkS")
 			(hide yes)
@@
 		)
 		(property "Value" "5.1k"
-			(at 0 1.43 270)
+			(at 0 1.43 -90)
 			(layer "F.Fab")
 			(effects
@@
 		)
 		(fp_text user "${REFERENCE}"
-			(at 0 0 270)
+			(at 0 0 -90)
 			(layer "F.Fab")
 			(effects
@@
 		)
 		(fp_text user "${REFERENCE}"
-			(at 0 -0.399999 279)
+			(at 0 -0.399999 -81)
 			(layer "F.Fab")
 			(effects
@@
 		(tags "resistor")
 		(property "Reference" "R5"
-			(at 0 -1.43 270)
+			(at 0 -1.43 -90)
 			(layer "F.SilkS")
 			(hide yes)
@@
 		)
 		(property "Value" "5.1k"
-			(at 0 1.43 270)
+			(at 0 1.43 -90)
 			(layer "F.Fab")
 			(effects
@@
 		)
 		(fp_text user "${REFERENCE}"
-			(at 0 0 270)
+			(at 0 0 -90)
 			(layer "F.Fab")
 			(effects
@@
 		)
 		(fp_text user "${REFERENCE}"
-			(at 0 -0.399999 189)
+			(at 0 -0.399999 -171)
 			(layer "F.Fab")
 			(effects
@@
 			)
 		)
-		(attr through_hole)
+		(attr through_hole exclude_from_pos_files exclude_from_bom)
 		(fp_circle
 			(center 0 -0.5)
@@
 			(size 1.29 1.29)
 			(layers "F.Paste")
-			(roundrect_rratio 0.193798)
+			(roundrect_rratio 0.1937976744)
 		)
 		(pad "" smd roundrect
@@
 			(size 1.29 1.29)
 			(layers "F.Paste")
-			(roundrect_rratio 0.193798)
+			(roundrect_rratio 0.1937976744)
 		)
 		(pad "" smd roundrect
@@
 			(size 1.29 1.29)
 			(layers "F.Paste")
-			(roundrect_rratio 0.193798)
+			(roundrect_rratio 0.1937976744)
 		)
 		(pad "" smd roundrect
@@
 			(size 1.29 1.29)
 			(layers "F.Paste")
-			(roundrect_rratio 0.193798)
+			(roundrect_rratio 0.1937976744)
 		)
 		(pad "1" smd roundrect
@@
 	)
 	(segment
-		(start 144.28452 85.148938)
-		(end 144.531299 84.389438)
-		(width 0.6)
-		(layer "F.Cu")
-		(net 2)
-	)
-	(segment
 		(start 128.034047 84.512444)
 		(end 128.70044 85.820309)
@@
 	)
 	(segment
-		(start 144.608436 85.784658)
-		(end 144.28452 85.148938)
-		(width 0.6)
-		(layer "F.Cu")
-		(net 2)
-	)
-	(segment
 		(start 142.011593 87.054525)
 		(end 141.555019 86.158454)
@@
 	)
 	(segment
+		(start 144.531299 85.131299)
+		(end 144.531299 84.389438)
+		(width 0.6)
+		(layer "F.Cu")
+		(net 2)
+	)
+	(segment
 		(start 142.662159 88.254249)
 		(end 142.459501 87.856512)
@@
 	)
 	(segment
+		(start 145 85.6)
+		(end 144.531299 85.131299)
+		(width 0.6)
+		(layer "F.Cu")
+		(net 2)
+	)
+	(segment
 		(start 138.019328 91.559839)
 		(end 136.90196 91.196784)
@@
 	)
 	(via
-		(at 144.608436 85.784658)
+		(at 145 85.6)
 		(size 0.6)
 		(drill 0.3)
@@
 		(layer "B.Cu")
 		(net 2)
-	)
-	(segment
-		(start 142.859939 85.216536)
-		(end 144.608436 85.784658)
-		(width 0.6)
-		(layer "B.Cu")
-		(net 2)
